File: KiCad/ArduFrauenfelderCNC.sch (KiCad schematic (older format))
At the start: 17 parts, among them IC1 MEGA8-P, J1 J1, J2 J2, Y1 16Mhz

Commit message: Update of schematic for KiCad (untested). Converted using eagle2kicad.ulp V1.1 and includes an initial commit of the .lib and .pro files.
Parts:
- added FRAME1: (no value), symbol FRAME_FRAME-A3
- added U$2: (no value), symbol SparkFun_OSHW-LOGO
Other:
- note added: "0.1-b3"
- note added: "Jamie Johnston"
